File: cpld_ex_100.sch (KiCad schematic (older format))
At the start: 83 parts, among them IC1 TBD62783A, IC2 SG-8002DC, IC3 MCP1826S, IC4 MCP1826S, IC5 MCP6022, J1 Jack-DC, SW1 SW_DIP_x08, SW2 SW_DIP_x08

Commit message: update
Parts:
- added CN1: Conn_02x05_Counter_Clockwise_MountingPin, symbol Connector_Generic:Conn_02x05_Odd_Even
- added unit 2 of IC5
- added unit 3 of IC5
- C1, C14, C2, C3, C4: symbol Device:C -> Device:C_Small
- J1: symbol Connector:Jack-DC -> Connector:Barrel_Jack_Switch
- R41, R43: value 10k -> 2.2k
- R42, R44: value 2.2k -> 10k
- VR1: symbol Device:R_Variable -> Device:R_POT
- gave numbers to parts that had none: 4
Connections:
- net D is gone; now on net A: C10.1, P3.13 (Pin_13)
- net A: now also C1.1, IC3.3 (VO)
- net B: now also IC5.3 (+)
- net GND: now also C1.2, C2.2, C3.2, C4.2, IC1.10 (GND), IC3.2 (GND), IC4.2 (GND), J1.2, J1.3, R22.2, R24.2, R28.2, R42.2, R44.2, TR1.1 (S), TR2.1 (S), VR1.3, CN1.10 (Pin_10), CN1.2 (Pin_2), IC5.4 (V-)
- net VDD: now also C2.1, IC1.9 (VCC), IC3.1 (VI), IC4.3 (VO), R25.1, R26.1, R27.1, CN1.4 (Pin_4)
- net at R21.1: now also VR1.2
- net at R21.2: now also IC5.5 (+)
- net at R22.1: now also R23.1, IC5.6 (-)
- net at R23.2: now also C14.1, IC5.7
- net at R24.1: now also C14.2
- net TDO: now reaches R27.2
- net TDO: now also P1.25 (Pin_25), CN1.3 (Pin_3)
- net TDI: now reaches R26.2
- net TDI: now also P1.23 (Pin_23), CN1.9 (Pin_9)
- net TMS: now reaches R25.2
- net TMS: now also P1.22 (Pin_22), CN1.5 (Pin_5)
- net TDK: now reaches R28.1
- net TDK: now also P1.24 (Pin_24), CN1.1 (Pin_1)
- net at R33.1: now also IC1.18 (O1)
- net at R33.2: now also LED5.3 (G), LED6.3 (G)
- net at R34.1: now also IC1.17 (O2)
- net at R34.2: now also LED5.2 (F), LED6.2 (F)
- net at R37.1: now also IC1.14 (O5)
- net at R37.2: now also LED5.8 (C), LED6.8 (C)
- net at R36.1: now also IC1.15 (O4)
- net at R36.2: now also LED5.5 (D), LED6.5 (D)
- net at R35.1: now also IC1.16 (O3)
- net at R35.2: now also LED5.4 (E), LED6.4 (E)
- net at R38.1: now also IC1.13 (O6)
- net at R38.2: now also LED5.9 (B), LED6.9 (B)
- net at R39.1: now also IC1.12 (O7)
- net at R39.2: now also LED5.10 (A), LED6.10 (A)
- net at R40.1: now also IC1.11 (O8)
- net at R40.2: now also LED5.7 (DP), LED6.7 (DP)
- net at R42.1: now also P4.21 (Pin_21), R41.1
- net at R41.2: now also TR1.2 (G)
- net at R43.1: now also P4.23 (Pin_23), R44.1
- net at R43.2: now also TR2.2 (G)
- net at VR1.1: now also IC5.1, IC5.2 (-)
- net at LED5.1 (CA): now also TR1.3 (D)
- net at LED6.1 (CA): now also TR2.3 (D)
- net at IC1.1 (I1): now also P4.17 (Pin_17)
- net at IC1.2 (I2): now also P4.16 (Pin_16)
- net at IC1.3 (I3): now also P4.15 (Pin_15)
- net at IC1.4 (I4): now also P4.14 (Pin_14)
- net at IC1.5 (I5): now also P4.13 (Pin_13)
- net at IC1.6 (I6): now also P4.12 (Pin_12)
- net at IC1.7 (I7): now also P4.11 (Pin_11)
- net at IC1.8 (I8): now also P4.10 (Pin_10)
- net at IC4.1 (VI): now also C3.1, J1.1, L1.1
- net at C4.1: now also L1.2, IC5.8 (V+)
Other:
- moved on the sheet: C1, C10, C11, C12, C13, C14, C15, C2, C3, C4, C5, C6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

Commit message: update
Connections:
- net at P1.12 (Pin_12): now also IC2.5 (OUT)
- net at P1.14 (Pin_14): no longer IC2.5 (OUT)
- no-connect marks 0 -> 44
Other:
- moved on the sheet: C1, C2, C3, C4, IC3, IC4, IC5C, J1, L1
